File: micro_redox_semi_split/micro_redox_semi_split.kicad_pcb (KiCad board)
At the start: 2 copper layers, 210.6 x 110.1 mm, 95 parts, among them J1 AVR-ISP-6, J2 PB6, J3 PC6, J4 Conn_01x01_Female, J5 PB0, J6 PE6, SW1 SW_SPST, SW10 SW_SPST, SW11 SW_SPST, SW12 SW_SPST, SW13 SW_SPST, SW14 SW_SPST, SW15 SW_SPST, SW16 SW_SPST, SW17 SW_SPST, SW18 SW_SPST, SW19 SW_SPST, SW2 SW_SPST, SW20 SW_SPST, SW21 SW_SPST, SW22 SW_SPST, SW23 SW_SPST, SW24 SW_SPST, SW25 SW_SPST, SW26 SW_SPST, SW27 SW_SPST, SW28 SW_SPST, SW29 SW_SPST, SW3 SW_SPST, SW30 SW_SPST, SW31 SW_SPST, SW32 SW_SPST, SW33 SW_SPST, SW34 SW_SPST, SW35 Rotary_Encoder_Switch, SW36 SW_Push, SW4 SW_SPST, SW5 SW_SPST, SW6 SW_SPST, SW7 SW_SPST, SW8 SW_SPST, SW9 SW_SPST, U1 PRTR5V0U2X, U2 ATmega32U4-AU, Y1 16MHz

Commit message: touch up and try some plugins
Parts:
- J4: value Conn_01x01_Female -> PC7
- moved C1 0.09 mm to (131.4, 89.3)
- moved D6 0.09 mm to (159.1, 76.4)
- moved SW31 0.09 mm to (85.7, 124.3)
- moved C6 0.09 mm to (128.6, 99.4)
- moved C7 0.09 mm to (140.3, 111.8)
- moved D30 0.09 mm to (239.5, 83.2)
- moved SW20 0.09 mm to (223.1, 65.4)
- moved D22 0.09 mm to (67.7, 92.0)
- moved SW2 0.09 mm to (74.6, 51.9)
- moved SW36 0.09 mm to (103.0, 118.3)
- moved D25 0.09 mm to (117.0, 114.4)
- moved C2 0.09 mm to (139.9, 89.3)
- moved D34 0.09 mm to (189.3, 113.0)
- moved SW5 0.09 mm to (123.8, 74.3)
- moved SW9 0.09 mm to (198.3, 51.9)
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Routing:
- net COL5: track 113.8 -> 120.5 mm
- net Net-(D15-Pad2): track 24.7 -> 30.2 mm
- net COL9: track 189.1 -> 193.3 mm
- net COL8: track 173.9 -> 175.3 mm
- net COL1: track 188.2 -> 189.5 mm
- net COL7: track 207.0 -> 206.1 mm
- net RST: track 84.6 -> 84.0 mm

Commit message: fixes for protos
Parts:
- added J7: PF7, Keebio-Parts:SinglePad, F.Cu at (133.6, 114.4)
- D1, D10, D11, D12, D13, D14, D15, D16, D17, D18, D19, D2, D20, D21, D22, D23, D24, D25, D26, D27, D28, D29, D3, D30, D31, D32, D33, D34, D35, D4, D5, D6, D7, D8, D9: footprint Diode_SMD:D_0805_2012Metric_Pad1.15x1.40mm_HandSolder -> Diode_SMD:D_SOD-123
- moved D20 3.07 mm to (230.2, 68.0)
- moved D30 2.57 mm to (237.0, 83.5)
- moved D10 2.48 mm to (224.4, 52.0)
- moved D35 2.36 mm to (146.1, 120.3), turned to 270 degrees
- moved D19 0.63 mm to (214.5, 69.1)
- moved D16 0.63 mm to (165.3, 91.5)
- moved D26 0.61 mm to (171.7, 107.4)
- moved D9 0.60 mm to (208.1, 53.4)
- moved D6 0.60 mm to (158.9, 75.8)
- moved D7 0.60 mm to (174.8, 66.9)
- moved D28 0.59 mm to (203.3, 89.5)
- moved D29 0.59 mm to (220.8, 85.0)
- moved D27 0.58 mm to (187.5, 98.4)
- moved D18 0.57 mm to (196.9, 73.8)
- moved D17 0.56 mm to (181.1, 82.7)
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Connections:
- D33 pad 1: Net-(D33-Pad1) -> ROW3
- D34 pad 1: Net-(D33-Pad1) -> ROW3
- D35 pad 1: Net-(D33-Pad1) -> ROW3
- SW35 pad S1: ROW3 -> COL5
- U2 pad 36: Net-(U2-Pad36) -> F-PF7
Routing:
- net ROW3: track 88.5 -> 154.2 mm
- net Net-(D33-Pad1): track 44.5 -> 0.00 mm
- net COL5: track 120.5 -> 131.2 mm, vias 0 -> 1
- net F-PF7: track 0.00 -> 5.18 mm
- net ROW1: track 216.7 -> 214.0 mm
- net ROW0: track 213.1 -> 215.3 mm
- net +5V: track 170.5 -> 172.5 mm
- net Net-(D10-Pad2): track 25.4 -> 23.9 mm
- net ROW2: track 238.5 -> 237.2 mm
- net Net-(D15-Pad2): track 30.2 -> 29.2 mm
- net Net-(D20-Pad2): track 25.4 -> 24.6 mm
- net Net-(D22-Pad2): track 24.9 -> 25.7 mm
- net Net-(D31-Pad2): track 28.0 -> 27.3 mm
- net Net-(D1-Pad2): track 24.9 -> 24.3 mm
- net Net-(D33-Pad2): track 26.5 -> 25.8 mm
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Other:
- board text added: "micro_redox_semi_split v0.second.try by makenova"
- board text removed: "trampstamp micro-redox v0.first.try by makenova"
