File: micro_redox_semi_split/micro_redox_semi_split.sch (KiCad schematic (older format))
At the start: 95 parts, among them J1 AVR-ISP-6, J2 Conn_01x01_Female, J3 Conn_01x01_Female, J4 Conn_01x01_Female, J5 Conn_01x01_Female, J6 Conn_01x01_Female, SW1 SW_SPST, SW10 SW_SPST, SW11 SW_SPST, SW12 SW_SPST, SW13 SW_SPST, SW14 SW_SPST, SW15 SW_SPST, SW16 SW_SPST, SW17 SW_SPST, SW18 SW_SPST, SW19 SW_SPST, SW2 SW_SPST, SW20 SW_SPST, SW21 SW_SPST, SW22 SW_SPST, SW23 SW_SPST, SW24 SW_SPST, SW25 SW_SPST, SW26 SW_SPST, SW27 SW_SPST, SW28 SW_SPST, SW29 SW_SPST, SW3 SW_SPST, SW30 SW_SPST, SW31 SW_SPST, SW32 SW_SPST, SW33 SW_SPST, SW34 SW_SPST, SW35 Rotary_Encoder_Switch, SW36 SW_Push, SW4 SW_SPST, SW5 SW_SPST, SW6 SW_SPST, SW7 SW_SPST, SW8 SW_SPST, SW9 SW_SPST, U1 PRTR5V0U2X, U2 ATmega32U4-AU, Y1 16MHz

Commit message: fixes for protos
Parts:
- added J7: PF7, Keebio-Parts:SinglePad, symbol Connector:Conn_01x01_Female
- D1, D10, D11, D12, D13, D14, D15, D16, D17, D18, D19, D2, D20, D21, D22, D23, D24, D25, D26, D27, D28, D29, D3, D30, D31, D32, D33, D34, D35, D4, D5, D6, D7, D8, D9: footprint Diode_SMD:D_0805_2012Metric_Pad1.15x1.40mm_HandSolder -> Diode_SMD:D_SOD-123
- J2: value Conn_01x01_Female -> PB6
- J3: value Conn_01x01_Female -> PC6
- J4: value Conn_01x01_Female -> PC7
- J5: value Conn_01x01_Female -> PB0
- J6: value Conn_01x01_Female -> PE6
Connections:
- net COL5: now also SW35.S1
- net ROW3: now also D33.1 (K), D34.1 (K), D35.1 (K); no longer SW35.S1
- net F-PF7: now reaches U2.36 (PF7)
- net F-PF7: now also J7.1 (Pin_1)
Other:
- moved on the sheet: J2, J3, J4, J5, J6
