File: micro_redox_split/micro_redox_split.kicad_pcb (KiCad board)
At the start: 2 copper layers, 99.8 x 89.8 mm, 20 parts, among them SW1 SW_SPST, U1 ProMicro, U2 TRRS

Commit message: fixes for protos
Routing:
- net S5: track 72.3 -> 74.9 mm
Other:
- board text added: "micro_redox_split v0.second.try by makenova"
- board text removed: "micro_redux v0.first.try by makenova"
Changed lines of the file:
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@@
     (thickness 1.6)
     (drawings 23)
-    (tracks 407)
+    (tracks 410)
     (zones 0)
     (modules 20)
@@
     (pad "" np_thru_hole circle (at -5.5 0 180) (size 1.7018 1.7018) (drill 1.7018) (layers *.Cu *.Mask))
   )
-  (gr_text JLCJLCJLCJLC (at 44.2595 139.7635) (layer F.Cu)
+  (gr_text JLCJLCJLCJLC (at 44.2595 139.7635) (layer F.SilkS)
     (effects (font (size 0.3 0.5) (thickness 0.0375)))
   )
-  (gr_text "micro_redux\nv0.first.try\nby makenova" (at 75.7555 135.382) (layer B.SilkS)
+  (gr_text "micro_redox_split\nv0.second.try\nby makenova" (at 75.7555 135.382) (layer B.SilkS)
     (effects (font (size 1.5 1.5) (thickness 0.3)) (justify mirror))
   )
-  (gr_text "micro_redux\nv0.first.try\nby makenova" (at 75.6285 135.382) (layer F.SilkS)
+  (gr_text "micro_redox_split\nv0.second.try\nby makenova" (at 75.6285 135.382) (layer F.SilkS)
     (effects (font (size 1.5 1.5) (thickness 0.3)))
   )
@@
   (segment (start 48.0695 125.73141) (end 50.80551 122.9954) (width 0.25) (layer F.Cu) (net 12))
   (segment (start 50.80551 122.9954) (end 50.80551 107.62699) (width 0.25) (layer F.Cu) (net 12))
-  (segment (start 50.80551 107.62699) (end 54.864 103.5685) (width 0.25) (layer F.Cu) (net 12))
+  (segment (start 54.891 103.5415) (end 54.61 103.8225) (width 0.25) (layer F.Cu) (net 12))
+  (segment (start 54.891 101.2635) (end 54.891 103.5415) (width 0.25) (layer F.Cu) (net 12))
+  (segment (start 54.61 103.8225) (end 54.864 103.5685) (width 0.25) (layer F.Cu) (net 12))
+  (segment (start 50.80551 107.62699) (end 54.61 103.8225) (width 0.25) (layer F.Cu) (net 12))
   (segment (start 61.441 116.7315) (end 61.441 118.2815) (width 0.25) (layer B.Cu) (net 13))
   (segment (start 54.5465 118.626) (end 54.891 118.2815) (width 0.25) (layer F.Cu) (net 13))
